Commit message: Fixed fingers

File: pepper_description/urdf/pepper1.0_generated_urdf/pepperGazebo.xacro (robot description, xacro)
@@ -56,18 +56,18 @@
             <joint>${side}Hand</joint>
             <mimicJoint>${side}Finger${num}1</mimicJoint>
-            <multiplier>-${PI/4}</multiplier>
-            <offset>${PI/4}</offset>
+            <multiplier>1</multiplier>
+            <offset>0</offset>
         </plugin>
         <plugin name="mimic_${side}Finger${num}2" filename="libroboticsgroup_gazebo_mimic_joint_plugin.so">
             <joint>${side}Hand</joint>
             <mimicJoint>${side}Finger${num}2</mimicJoint>
-            <multiplier>-${PI/4}</multiplier>
-            <offset>${PI/4}</offset>
+            <multiplier>1</multiplier>
+            <offset>0</offset>
         </plugin>
         <plugin name="mimic_${side}Finger${num}3" filename="libroboticsgroup_gazebo_mimic_joint_plugin.so">
             <joint>${side}Hand</joint>
             <mimicJoint>${side}Finger${num}3</mimicJoint>
-            <multiplier>-${PI/4}</multiplier>
-            <offset>${PI/4}</offset>
+            <multiplier>1</multiplier>
+            <offset>0</offset>
         </plugin>
     </xacro:macro>
@@ -77,12 +77,12 @@
             <joint>${side}Hand</joint>
             <mimicJoint>${side}Thumb1</mimicJoint>
-            <multiplier>-${PI/4}</multiplier>
-            <offset>${PI/4}</offset>
+            <multiplier>1</multiplier>
+            <offset>0</offset>
         </plugin>
         <plugin name="${side}Thumb2" filename="libroboticsgroup_gazebo_mimic_joint_plugin.so">
             <joint>${side}Hand</joint>
             <mimicJoint>${side}Thumb2</mimicJoint>
-            <multiplier>-${PI/4}</multiplier>
-            <offset>${PI/4}</offset>
+            <multiplier>1</multiplier>
+            <offset>0</offset>
         </plugin>
     </xacro:macro>
@@ -103,6 +103,7 @@
         <xacro:ThumbMimics side="L"/>
         <xacro:ThumbMimics side="R"/>
+<!--
         <xacro:DisabledLinks side="L" side_small="l"/>
-        <xacro:DisabledLinks side="R" side_small="r"/>
+        <xacro:DisabledLinks side="R" side_small="r"/>  -->
     </gazebo>
     <!-- END OF GAZEBO ROS CONTROL PLUGIN -->
@@ -173,5 +174,5 @@
         <mu2>0.5</mu2>
         <selfCollide>false</selfCollide>
-        <turnGravityOff>true</turnGravityOff>
+        <turnGravityOff>false</turnGravityOff>
     </gazebo>
     <gazebo reference="RShoulder">
@@ -209,5 +210,5 @@
         <mu2>0.5</mu2>
         <selfCollide>false</selfCollide>
-        <turnGravityOff>true</turnGravityOff>
+        <turnGravityOff>false</turnGravityOff>
     </gazebo>
     <gazebo reference="LFinger11_link">
@@ -344,5 +345,5 @@
         <mu2>0.5</mu2>
         <selfCollide>false</selfCollide>
-        <turnGravityOff>true</turnGravityOff>
+        <turnGravityOff>false</turnGravityOff>
     </gazebo>
     <gazebo reference="RFinger12_link">
@@ -350,5 +351,5 @@
         <mu2>0.5</mu2>
         <selfCollide>false</selfCollide>
-        <turnGravityOff>true</turnGravityOff>
+        <turnGravityOff>false</turnGravityOff>
     </gazebo>
     <gazebo reference="RFinger13_link">
@@ -356,5 +357,5 @@
         <mu2>0.5</mu2>
         <selfCollide>false</selfCollide>
-        <turnGravityOff>true</turnGravityOff>
+        <turnGravityOff>false</turnGravityOff>
     </gazebo>
     <gazebo reference="RFinger21_link">
@@ -362,5 +363,5 @@
         <mu2>0.5</mu2>
         <selfCollide>false</selfCollide>
-        <turnGravityOff>true</turnGravityOff>
+        <turnGravityOff>false</turnGravityOff>
     </gazebo>
     <gazebo reference="RFinger22_link">
@@ -368,5 +369,5 @@
         <mu2>0.5</mu2>
         <selfCollide>false</selfCollide>
-        <turnGravityOff>true</turnGravityOff>
+        <turnGravityOff>false</turnGravityOff>
     </gazebo>
     <gazebo reference="RFinger23_link">
@@ -374,5 +375,5 @@
         <mu2>0.5</mu2>
         <selfCollide>false</selfCollide>
-        <turnGravityOff>true</turnGravityOff>
+        <turnGravityOff>false</turnGravityOff>
     </gazebo>
     <gazebo reference="RFinger31_link">
@@ -380,5 +381,5 @@
         <mu2>0.5</mu2>
         <selfCollide>false</selfCollide>
-        <turnGravityOff>true</turnGravityOff>
+        <turnGravityOff>false</turnGravityOff>
     </gazebo>
     <gazebo reference="RFinger32_link">
@@ -386,5 +387,5 @@
         <mu2>0.5</mu2>
         <selfCollide>false</selfCollide>
-        <turnGravityOff>true</turnGravityOff>
+        <turnGravityOff>false</turnGravityOff>
     </gazebo>
     <gazebo reference="RFinger33_link">
@@ -392,5 +393,5 @@
         <mu2>0.5</mu2>
         <selfCollide>false</selfCollide>
-        <turnGravityOff>true</turnGravityOff>
+        <turnGravityOff>false</turnGravityOff>
     </gazebo>
     <gazebo reference="RFinger41_link">
@@ -398,5 +399,5 @@
         <mu2>0.5</mu2>
         <selfCollide>false</selfCollide>
-        <turnGravityOff>true</turnGravityOff>
+        <turnGravityOff>false</turnGravityOff>
     </gazebo>
     <gazebo reference="RFinger42_link">
@@ -404,5 +405,5 @@
         <mu2>0.5</mu2>
         <selfCollide>false</selfCollide>
-        <turnGravityOff>true</turnGravityOff>
+        <turnGravityOff>false</turnGravityOff>
     </gazebo>
     <gazebo reference="RFinger43_link">
@@ -410,5 +411,5 @@
         <mu2>0.5</mu2>
         <selfCollide>false</selfCollide>
-        <turnGravityOff>true</turnGravityOff>
+        <turnGravityOff>false</turnGravityOff>
     </gazebo>
     <gazebo reference="RThumb1_link">
@@ -416,5 +417,5 @@
         <mu2>0.5</mu2>
         <selfCollide>false</selfCollide>
-        <turnGravityOff>true</turnGravityOff>
+        <turnGravityOff>false</turnGravityOff>
     </gazebo>
     <gazebo reference="RThumb2_link">
@@ -422,5 +423,5 @@
         <mu2>0.5</mu2>
         <selfCollide>false</selfCollide>
-        <turnGravityOff>true</turnGravityOff>
+        <turnGravityOff>false</turnGravityOff>
     </gazebo>
 <!--

File: pepper_description/urdf/pepper1.0_generated_urdf/pepper_arms.xacro (robot description, xacro)
@@ -74,5 +74,5 @@
 		<inertial>
 			<mass value="0.27555"/>
-			<inertia ixx="0.000151643" ixy="1.06629e-05" ixz="2.89509e-06" iyy="0.000431099" iyz="-3.13715e-06" izz="0.000456172"/>
+			<inertia ixx="0.00156513" ixy="-1.47517e-05" ixz="-6.05746e-05" iyy="0.00173219" iyz="1.7619e-07" izz="0.000273081"/>
 			<origin rpy="0 0 0" xyz="0.03536 -0.00072 -0.00207"/>
 		</inertial>
@@ -88,6 +88,6 @@
 	<link name="l_gripper">
 		<inertial>
-			<mass value="2e-06"/>
-			<inertia ixx="1.1e-09" ixy="0" ixz="0" iyy="1.1e-09" iyz="0" izz="1.1e-09"/>
+			<mass value="0.0016579"/>
+			<inertia ixx="0.00156513" ixy="-1.47517e-05" ixz="-6.05746e-05" iyy="0.00173219" iyz="1.7619e-07" izz="0.000273081"/>
 		</inertial>
 	</link>
@@ -162,5 +162,5 @@
 		<inertial>
 			<mass value="0.27555"/>
-			<inertia ixx="0.000151643" ixy="-1.06629e-05" ixz="2.89509e-06" iyy="0.000431099" iyz="3.13715e-06" izz="0.000456172"/>
+			<inertia ixx="0.00156513" ixy="-1.47517e-05" ixz="-6.05746e-05" iyy="0.00173219" iyz="1.7619e-07" izz="0.000273081"/>
 			<origin rpy="0 0 0" xyz="0.03536 0.00072 -0.00207"/>
 		</inertial>
@@ -176,6 +176,6 @@
 	<link name="r_gripper">
 		<inertial>
-			<mass value="2e-06"/>
-			<inertia ixx="1.1e-09" ixy="0" ixz="0" iyy="1.1e-09" iyz="0" izz="1.1e-09"/>
+			<mass value="0.0016579"/>
+			<inertia ixx="0.00156513" ixy="-1.47517e-05" ixz="-6.05746e-05" iyy="0.00173219" iyz="1.7619e-07" izz="0.000273081"/>
 		</inertial>
 	</link>

File: pepper_description/urdf/pepper1.0_generated_urdf/pepper_fingers.xacro (robot description, xacro)
@@ -6,6 +6,6 @@
 	<link name="RFinger41_link">
 		<inertial>
-			<mass value="2e-06"/>
-			<inertia ixx="1.1e-09" ixy="0" ixz="0" iyy="1.1e-09" iyz="0" izz="1.1e-09"/>
+			<mass value="2e-03"/>
+			<inertia ixx="0.001" ixy="0" ixz="0" iyy="0.001" iyz="0" izz="0.001"/>
 		</inertial>
 		<xacro:insert_visu_RFinger41_link/>
@@ -16,10 +16,10 @@
 		<origin rpy="1.74402 1.04064 -0.0683394" xyz="0.074 -0.0309 0"/>
 		<axis xyz="0 0 1.0"/>
-		<mimic joint="RHand" multiplier="0.872665" offset="0"/>
+		<mimic joint="RHand" multiplier="1" offset="0"/>
 	</joint>
 	<link name="LFinger42_link">
 		<inertial>
-			<mass value="2e-06"/>
-			<inertia ixx="1.1e-09" ixy="0" ixz="0" iyy="1.1e-09" iyz="0" izz="1.1e-09"/>
+			<mass value="2e-03"/>
+			<inertia ixx="0.001" ixy="0" ixz="0" iyy="0.001" iyz="0" izz="0.001"/>
 		</inertial>
 		<xacro:insert_visu_LFinger42_link/>
@@ -30,10 +30,10 @@
 		<origin rpy="0 0 -1.0472" xyz="0.018 0 0"/>
 		<axis xyz="0 0 1.0"/>
-		<mimic joint="LHand" multiplier="0.872665" offset="0"/>
+		<mimic joint="LHand" multiplier="1" offset="0"/>
 	</joint>
 	<link name="RFinger12_link">
 		<inertial>
-			<mass value="2e-06"/>
-			<inertia ixx="1.1e-09" ixy="0" ixz="0" iyy="1.1e-09" iyz="0" izz="1.1e-09"/>
+			<mass value="2e-03"/>
+			<inertia ixx="0.001" ixy="0" ixz="0" iyy="0.001" iyz="0" izz="0.001"/>
 		</inertial>
 		<xacro:insert_visu_RFinger12_link/>
@@ -44,10 +44,10 @@
 		<origin rpy="0 0 -1.0472" xyz="0.018 0 0"/>
 		<axis xyz="0 0 1.0"/>
-		<mimic joint="RHand" multiplier="0.872665" offset="0"/>
+		<mimic joint="RHand" multiplier="1" offset="0"/>
 	</joint>
 	<link name="LFinger33_link">
 		<inertial>
-			<mass value="2e-06"/>
-			<inertia ixx="1.1e-09" ixy="0" ixz="0" iyy="1.1e-09" iyz="0" izz="1.1e-09"/>
+			<mass value="2e-03"/>
+			<inertia ixx="0.001" ixy="0" ixz="0" iyy="0.001" iyz="0" izz="0.001"/>
 		</inertial>
 		<xacro:insert_visu_LFinger33_link/>
@@ -58,10 +58,10 @@
 		<origin rpy="0 0 -1.0472" xyz="0.018 0 0"/>
 		<axis xyz="0 0 1.0"/>
-		<mimic joint="LHand" multiplier="0.872665" offset="0"/>
+		<mimic joint="LHand" multiplier="1" offset="0"/>
 	</joint>
 	<link name="RFinger31_link">
 		<inertial>
-			<mass value="2e-06"/>
-			<inertia ixx="1.1e-09" ixy="0" ixz="0" iyy="1.1e-09" iyz="0" izz="1.1e-09"/>
+			<mass value="2e-03"/>
+			<inertia ixx="0.001" ixy="0" ixz="0" iyy="0.001" iyz="0" izz="0.001"/>
 		</inertial>
 		<xacro:insert_visu_RFinger31_link/>
@@ -72,10 +72,10 @@
 		<origin rpy="1.67523 1.04483 0.029316" xyz="0.0833 -0.0123 0.004"/>
 		<axis xyz="0 0 1.0"/>
-		<mimic joint="RHand" multiplier="0.872665" offset="0"/>
+		<mimic joint="RHand" multiplier="1" offset="0"/>
 	</joint>
 	<link name="LFinger21_link">
 		<inertial>
-			<mass value="2e-06"/>
-			<inertia ixx="1.1e-09" ixy="0" ixz="0" iyy="1.1e-09" iyz="0" izz="1.1e-09"/>
+			<mass value="2e-03"/>
+			<inertia ixx="0.001" ixy="0" ixz="0" iyy="0.001" iyz="0" izz="0.001"/>
 		</inertial>
 		<xacro:insert_visu_LFinger21_link/>
@@ -86,10 +86,10 @@
 		<origin rpy="1.5708 1.0472 -0.061086" xyz="0.0873 -0.0073 0.006"/>
 		<axis xyz="0 0 1.0"/>
-		<mimic joint="LHand" multiplier="0.872665" offset="0"/>
+		<mimic joint="LHand" multiplier="1" offset="0"/>
 	</joint>
 	<link name="RFinger32_link">
 		<inertial>
-			<mass value="2e-06"/>
-			<inertia ixx="1.1e-09" ixy="0" ixz="0" iyy="1.1e-09" iyz="0" izz="1.1e-09"/>
+			<mass value="2e-03"/>
+			<inertia ixx="0.001" ixy="0" ixz="0" iyy="0.001" iyz="0" izz="0.001"/>
 		</inertial>
 		<xacro:insert_visu_RFinger32_link/>
@@ -100,10 +100,10 @@
 		<origin rpy="0 0 -1.0472" xyz="0.018 0 0"/>
 		<axis xyz="0 0 1.0"/>
-		<mimic joint="RHand" multiplier="0.872665" offset="0"/>
+		<mimic joint="RHand" multiplier="1" offset="0"/>
 	</joint>
 	<link name="LFinger13_link">
 		<inertial>
-			<mass value="2e-06"/>
-			<inertia ixx="1.1e-09" ixy="0" ixz="0" iyy="1.1e-09" iyz="0" izz="1.1e-09"/>
+			<mass value="2e-03"/>
+			<inertia ixx="0.001" ixy="0" ixz="0" iyy="0.001" iyz="0" izz="0.001"/>
 		</inertial>
 		<xacro:insert_visu_LFinger13_link/>
@@ -114,10 +114,10 @@
 		<origin rpy="0 0 -1.0472" xyz="0.018 0 0"/>
 		<axis xyz="0 0 1.0"/>
-		<mimic joint="LHand" multiplier="0.872665" offset="0"/>
+		<mimic joint="LHand" multiplier="1" offset="0"/>
 	</joint>
 	<link name="LFinger32_link">
 		<inertial>
-			<mass value="2e-06"/>
-			<inertia ixx="1.1e-09" ixy="0" ixz="0" iyy="1.1e-09" iyz="0" izz="1.1e-09"/>
+			<mass value="2e-03"/>
+			<inertia ixx="0.001" ixy="0" ixz="0" iyy="0.001" iyz="0" izz="0.001"/>
 		</inertial>
 		<xacro:insert_visu_LFinger32_link/>
@@ -128,10 +128,10 @@
 		<origin rpy="0 0 -1.0472" xyz="0.018 0 0"/>
 		<axis xyz="0 0 1.0"/>
-		<mimic joint="LHand" multiplier="0.872665" offset="0"/>
+		<mimic joint="LHand" multiplier="1" offset="0"/>
 	</joint>
 	<link name="LFinger11_link">
 		<inertial>
-			<mass value="2e-06"/>
-			<inertia ixx="1.1e-09" ixy="0" ixz="0" iyy="1.1e-09" iyz="0" izz="1.1e-09"/>
+			<mass value="2e-03"/>
+			<inertia ixx="0.001" ixy="0" ixz="0" iyy="0.001" iyz="0" izz="0.001"/>
 		</inertial>
 		<xacro:insert_visu_LFinger11_link/>
@@ -142,10 +142,10 @@
 		<origin rpy="1.74402 1.04064 -0.0334335" xyz="0.0821 -0.0268 0.004"/>
 		<axis xyz="0 0 1.0"/>
-		<mimic joint="LHand" multiplier="0.872665" offset="0"/>
+		<mimic joint="LHand" multiplier="1" offset="0"/>
 	</joint>
 	<link name="RFinger22_link">
 		<inertial>
-			<mass value="2e-06"/>
-			<inertia ixx="1.1e-09" ixy="0" ixz="0" iyy="1.1e-09" iyz="0" izz="1.1e-09"/>
+			<mass value="2e-03"/>
+			<inertia ixx="0.001" ixy="0" ixz="0" iyy="0.001" iyz="0" izz="0.001"/>
 		</inertial>
 		<xacro:insert_visu_RFinger22_link/>
@@ -156,10 +156,10 @@
 		<origin rpy="0 0 -1.0472" xyz="0.018 0 0"/>
 		<axis xyz="0 0 1.0"/>
-		<mimic joint="RHand" multiplier="0.872665" offset="0"/>
+		<mimic joint="RHand" multiplier="1" offset="0"/>
 	</joint>
 	<link name="RFinger13_link">
 		<inertial>
-			<mass value="2e-06"/>
-			<inertia ixx="1.1e-09" ixy="0" ixz="0" iyy="1.1e-09" iyz="0" izz="1.1e-09"/>
+			<mass value="2e-03"/>
+			<inertia ixx="0.001" ixy="0" ixz="0" iyy="0.001" iyz="0" izz="0.001"/>
 		</inertial>
 		<xacro:insert_visu_RFinger13_link/>
@@ -170,10 +170,10 @@
 		<origin rpy="0 0 -1.0472" xyz="0.018 0 0"/>
 		<axis xyz="0 0 1.0"/>
-		<mimic joint="RHand" multiplier="0.872665" offset="0"/>
+		<mimic joint="RHand" multiplier="1" offset="0"/>
 	</joint>
 	<link name="LFinger22_link">
 		<inertial>
-			<mass value="2e-06"/>
-			<inertia ixx="1.1e-09" ixy="0" ixz="0" iyy="1.1e-09" iyz="0" izz="1.1e-09"/>
+			<mass value="2e-03"/>
+			<inertia ixx="0.001" ixy="0" ixz="0" iyy="0.001" iyz="0" izz="0.001"/>
 		</inertial>
 		<xacro:insert_visu_LFinger22_link/>
@@ -184,10 +184,10 @@
 		<origin rpy="0 0 -1.0472" xyz="0.018 0 0"/>
 		<axis xyz="0 0 1.0"/>
-		<mimic joint="LHand" multiplier="0.872665" offset="0"/>
+		<mimic joint="LHand" multiplier="1" offset="0"/>
 	</joint>
 	<link name="RFinger21_link">
 		<inertial>
-			<mass value="2e-06"/>
-			<inertia ixx="1.1e-09" ixy="0" ixz="0" iyy="1.1e-09" iyz="0" izz="1.1e-09"/>
+			<mass value="2e-03"/>
+			<inertia ixx="0.001" ixy="0" ixz="0" iyy="0.001" iyz="0" izz="0.001"/>
 		</inertial>
 		<xacro:insert_visu_RFinger21_link/>
@@ -198,10 +198,10 @@
 		<origin rpy="1.5708 1.0472 0.061086" xyz="0.0873 0.0073 0.006"/>
 		<axis xyz="0 0 1.0"/>
-		<mimic joint="RHand" multiplier="0.872665" offset="0"/>
+		<mimic joint="RHand" multiplier="1" offset="0"/>
 	</joint>
 	<link name="LFinger41_link">
 		<inertial>
-			<mass value="2e-06"/>
-			<inertia ixx="1.1e-09" ixy="0" ixz="0" iyy="1.1e-09" iyz="0" izz="1.1e-09"/>
+			<mass value="2e-03"/>
+			<inertia ixx="0.001" ixy="0" ixz="0" iyy="0.001" iyz="0" izz="0.001"/>
 		</inertial>
 		<xacro:insert_visu_LFinger41_link/>
@@ -210,12 +210,12 @@
 		<parent link="l_wrist"/>
 		<child link="LFinger41_link"/>
-		<origin rpy="1.39757 1.04064 0.0683394" xyz="0.074 0.0309 0"/>
-		<axis xyz="0 0 1.0"/>
-		<mimic joint="LHand" multiplier="0.872665" offset="0"/>
+		<origin rpy="1.74402 1.04064 0.0683394" xyz="0.074 0.0309 0"/>
+		<axis xyz="0 0 1.0"/>
+		<mimic joint="LHand" multiplier="1" offset="0"/>
 	</joint>
 	<link name="LFinger12_link">
 		<inertial>
-			<mass value="2e-06"/>
-			<inertia ixx="1.1e-09" ixy="0" ixz="0" iyy="1.1e-09" iyz="0" izz="1.1e-09"/>
+			<mass value="2e-03"/>
+			<inertia ixx="0.001" ixy="0" ixz="0" iyy="0.001" iyz="0" izz="0.001"/>
 		</inertial>
 		<xacro:insert_visu_LFinger12_link/>
@@ -226,10 +226,10 @@
 		<origin rpy="0 0 -1.0472" xyz="0.018 0 0"/>
 		<axis xyz="0 0 1.0"/>
-		<mimic joint="LHand" multiplier="0.872665" offset="0"/>
+		<mimic joint="LHand" multiplier="1" offset="0"/>
 	</joint>
 	<link name="RFinger23_link">
 		<inertial>
-			<mass value="2e-06"/>
-			<inertia ixx="1.1e-09" ixy="0" ixz="0" iyy="1.1e-09" iyz="0" izz="1.1e-09"/>
+			<mass value="2e-03"/>
+			<inertia ixx="0.001" ixy="0" ixz="0" iyy="0.001" iyz="0" izz="0.001"/>
 		</inertial>
 		<xacro:insert_visu_RFinger23_link/>
@@ -240,10 +240,10 @@
 		<origin rpy="0 0 -1.0472" xyz="0.018 0 0"/>
 		<axis xyz="0 0 1.0"/>
-		<mimic joint="RHand" multiplier="0.872665" offset="0"/>
+		<mimic joint="RHand" multiplier="1" offset="0"/>
 	</joint>
 	<link name="RFinger11_link">
 		<inertial>
-			<mass value="2e-06"/>
-			<inertia ixx="1.1e-09" ixy="0" ixz="0" iyy="1.1e-09" iyz="0" izz="1.1e-09"/>
+			<mass value="2e-03"/>
+			<inertia ixx="0.001" ixy="0" ixz="0" iyy="0.001" iyz="0" izz="0.001"/>
 		</inertial>
 		<xacro:insert_visu_RFinger11_link/>
@@ -254,10 +254,10 @@
 		<origin rpy="1.39757 1.04064 0.0334335" xyz="0.0821 0.0268 0.004"/>
 		<axis xyz="0 0 1.0"/>
-		<mimic joint="RHand" multiplier="0.872665" offset="0"/>
+		<mimic joint="RHand" multiplier="1" offset="0"/>
 	</joint>
 	<link name="LFinger23_link">
 		<inertial>
-			<mass value="2e-06"/>
-			<inertia ixx="1.1e-09" ixy="0" ixz="0" iyy="1.1e-09" iyz="0" izz="1.1e-09"/>
+			<mass value="2e-03"/>
+			<inertia ixx="0.001" ixy="0" ixz="0" iyy="0.001" iyz="0" izz="0.001"/>
 		</inertial>
 		<xacro:insert_visu_LFinger23_link/>
@@ -268,10 +268,10 @@
 		<origin rpy="0 0 -1.0472" xyz="0.018 0 0"/>
 		<axis xyz="0 0 1.0"/>
-		<mimic joint="LHand" multiplier="0.872665" offset="0"/>
+		<mimic joint="LHand" multiplier="1" offset="0"/>
 	</joint>
 	<link name="LFinger43_link">
 		<inertial>
-			<mass value="2e-06"/>
-			<inertia ixx="1.1e-09" ixy="0" ixz="0" iyy="1.1e-09" iyz="0" izz="1.1e-09"/>
+			<mass value="2e-03"/>
+			<inertia ixx="0.001" ixy="0" ixz="0" iyy="0.001" iyz="0" izz="0.001"/>
 		</inertial>
 		<xacro:insert_visu_LFinger43_link/>
@@ -282,10 +282,10 @@
 		<origin rpy="0 0 -1.0472" xyz="0.018 0 0"/>
 		<axis xyz="0 0 1.0"/>
-		<mimic joint="LHand" multiplier="0.872665" offset="0"/>
+		<mimic joint="LHand" multiplier="1" offset="0"/>
 	</joint>
 	<link name="RFinger43_link">
 		<inertial>
-			<mass value="2e-06"/>
-			<inertia ixx="1.1e-09" ixy="0" ixz="0" iyy="1.1e-09" iyz="0" izz="1.1e-09"/>
+			<mass value="2e-03"/>
+			<inertia ixx="0.001" ixy="0" ixz="0" iyy="0.001" iyz="0" izz="0.001"/>
 		</inertial>
 		<xacro:insert_visu_RFinger43_link/>
@@ -296,10 +296,10 @@
 		<origin rpy="0 0 -1.0472" xyz="0.018 0 0"/>
 		<axis xyz="0 0 1.0"/>
-		<mimic joint="RHand" multiplier="0.872665" offset="0"/>
+		<mimic joint="RHand" multiplier="1" offset="0"/>
 	</joint>
 	<link name="RFinger42_link">
 		<inertial>
-			<mass value="2e-06"/>
-			<inertia ixx="1.1e-09" ixy="0" ixz="0" iyy="1.1e-09" iyz="0" izz="1.1e-09"/>
+			<mass value="2e-03"/>
+			<inertia ixx="0.001" ixy="0" ixz="0" iyy="0.001" iyz="0" izz="0.001"/>
 		</inertial>
 		<xacro:insert_visu_RFinger42_link/>
@@ -310,10 +310,10 @@
 		<origin rpy="0 0 -1.0472" xyz="0.018 0 0"/>
 		<axis xyz="0 0 1.0"/>
-		<mimic joint="RHand" multiplier="0.872665" offset="0"/>
+		<mimic joint="RHand" multiplier="1" offset="0"/>
 	</joint>
 	<link name="LFinger31_link">
 		<inertial>
-			<mass value="2e-06"/>
-			<inertia ixx="1.1e-09" ixy="0" ixz="0" iyy="1.1e-09" iyz="0" izz="1.1e-09"/>
+			<mass value="2e-03"/>
+			<inertia ixx="0.001" ixy="0" ixz="0" iyy="0.001" iyz="0" izz="0.001"/>
 		</inertial>
 		<xacro:insert_visu_LFinger31_link/>
@@ -322,12 +322,12 @@
 		<parent link="l_wrist"/>
 		<child link="LFinger31_link"/>
-		<origin rpy="1.46636 1.04483 -0.029314" xyz="0.0833 0.0123 0.004"/>
-		<axis xyz="0 0 1.0"/>
-		<mimic joint="LHand" multiplier="0.872665" offset="0"/>
+		<origin rpy="1.67523 1.04483 -0.029316" xyz="0.0833 0.0123 0.004"/>
+		<axis xyz="0 0 1.0"/>
+		<mimic joint="LHand" multiplier="1" offset="0"/>
 	</joint>
 	<link name="RFinger33_link">
 		<inertial>
-			<mass value="2e-06"/>
-			<inertia ixx="1.1e-09" ixy="0" ixz="0" iyy="1.1e-09" iyz="0" izz="1.1e-09"/>
+			<mass value="2e-03"/>
+			<inertia ixx="0.001" ixy="0" ixz="0" iyy="0.001" iyz="0" izz="0.001"/>
 		</inertial>
 		<xacro:insert_visu_RFinger33_link/>
@@ -338,10 +338,10 @@
 		<origin rpy="0 0 -1.0472" xyz="0.018 0 0"/>
 		<axis xyz="0 0 1.0"/>
-		<mimic joint="RHand" multiplier="0.872665" offset="0"/>
+		<mimic joint="RHand" multiplier="1" offset="0"/>
 	</joint>
 	<link name="LThumb1_link">
 		<inertial>
-			<mass value="2e-06"/>
-			<inertia ixx="1.1e-09" ixy="0" ixz="0" iyy="1.1e-09" iyz="0" izz="1.1e-09"/>
+			<mass value="2e-03"/>
+			<inertia ixx="0.001" ixy="0" ixz="0" iyy="0.001" iyz="0" izz="0.001"/>
 		</inertial>
 		<xacro:insert_visu_LThumb1_link/>
@@ -350,12 +350,12 @@
 		<parent link="l_wrist"/>
 		<child link="LThumb1_link"/>
-		<origin rpy="-1.95836 0.60626 0.533978" xyz="0.0482 -0.0357 -0.0199"/>
-		<axis xyz="0 0 1.0"/>
-		<mimic joint="LHand" multiplier="0.872665" offset="0"/>
+		<origin rpy="-1.18323 0.60626 0.533978" xyz="0.0482 -0.0357 -0.0199"/>
+		<axis xyz="0 0 1.0"/>
+		<mimic joint="LHand" multiplier="1" offset="0"/>
 	</joint>
 	<link name="RThumb2_link">
 		<inertial>
-			<mass value="2e-06"/>
-			<inertia ixx="1.1e-09" ixy="0" ixz="0" iyy="1.1e-09" iyz="0" izz="1.1e-09"/>
+			<mass value="2e-03"/>
+			<inertia ixx="0.001" ixy="0" ixz="0" iyy="0.001" iyz="0" izz="0.001"/>
 		</inertial>
 		<xacro:insert_visu_RThumb2_link/>
@@ -366,10 +366,10 @@
 		<origin rpy="0 0 -1.0472" xyz="0.022 0 0"/>
 		<axis xyz="0 0 1.0"/>
-		<mimic joint="RHand" multiplier="0.872665" offset="0"/>
+		<mimic joint="RHand" multiplier="1" offset="0"/>
 	</joint>
 	<link name="RThumb1_link">
 		<inertial>
-			<mass value="2e-06"/>
-			<inertia ixx="1.1e-09" ixy="0" ixz="0" iyy="1.1e-09" iyz="0" izz="1.1e-09"/>
+			<mass value="2e-03"/>
+			<inertia ixx="0.001" ixy="0" ixz="0" iyy="0.001" iyz="0" izz="0.001"/>
 		</inertial>
 		<xacro:insert_visu_RThumb1_link/>
@@ -380,10 +380,10 @@
 		<origin rpy="-1.18323 0.60626 -0.533978" xyz="0.0482 0.0357 -0.0199"/>
 		<axis xyz="0 0 1.0"/>
-		<mimic joint="RHand" multiplier="0.872665" offset="0"/>
+		<mimic joint="RHand" multiplier="1" offset="0"/>
 	</joint>
 	<link name="LThumb2_link">
 		<inertial>
-			<mass value="2e-06"/>
-			<inertia ixx="1.1e-09" ixy="0" ixz="0" iyy="1.1e-09" iyz="0" izz="1.1e-09"/>
+			<mass value="2e-03"/>
+			<inertia ixx="0.001" ixy="0" ixz="0" iyy="0.001" iyz="0" izz="0.001"/>
 		</inertial>
 		<xacro:insert_visu_LThumb2_link/>
@@ -394,5 +394,5 @@
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