Commit message: Better arm simulation and moveit configuration

File: pepper_description/urdf/pepper1.0_generated_urdf/pepper_arms.xacro (robot description, xacro)
@@ -14,5 +14,5 @@
 		<inertial>
 			<mass value="0.3125"/>
-			<inertia ixx="0.000361198" ixy="-1.98347e-06" ixz="6.35907e-07" iyy="0.000137229" iyz="-5.68878e-06" izz="0.000399194"/>
+			<inertia ixx="0.000361198" ixy="0" ixz="0" iyy="0.000137229" iyz="0" izz="0.000399194"/>
 			<origin rpy="0 0 0" xyz="0.00018 -0.01856 0.00099"/>
 		</inertial>
@@ -29,5 +29,5 @@
 		<inertial>
 			<mass value="0.50527"/>
-			<inertia ixx="0.000500872" ixy="-3.55918e-05" ixz="8.51263e-05" iyy="0.00126284" iyz="9.06813e-06" izz="0.00115718"/>
+			<inertia ixx="0.000500872" ixy="0" ixz="0" iyy="0.00126284" iyz="0" izz="0.00115718"/>
 			<origin rpy="0 0 0" xyz="0.08151 0.01284 -0.01017"/>
 		</inertial>
@@ -44,5 +44,5 @@
 		<inertial>
 			<mass value="0.27495"/>
-			<inertia ixx="0.000122971" ixy="9.86024e-07" ixz="-2.55838e-05" iyy="0.000331766" iyz="-1.98925e-06" izz="0.000303047"/>
+			<inertia ixx="0.000122971" ixy="0" ixz="0" iyy="0.000331766" iyz="0" izz="0.000303047"/>
 			<origin rpy="0 0 0" xyz="-0.02297 -0.00019 0.00119"/>
 		</inertial>
@@ -59,5 +59,5 @@
 		<inertial>
 			<mass value="0.16579"/>
-			<inertia ixx="0.00156513" ixy="1.47517e-05" ixz="-6.05746e-05" iyy="0.00173219" iyz="-1.7619e-07" izz="0.000273081"/>
+			<inertia ixx="0.00156513" ixy="0" ixz="0" iyy="0.00173219" iyz="0" izz="0.000273081"/>
 			<origin rpy="0 0 0" xyz="0.0593 0.00271 -0.01014"/>
 		</inertial>
@@ -73,6 +73,6 @@
 	<link name="l_wrist">
 		<inertial>
-			<mass value="0.27555"/>
-			<inertia ixx="0.00156513" ixy="-1.47517e-05" ixz="-6.05746e-05" iyy="0.00173219" iyz="1.7619e-07" izz="0.000273081"/>
+			<mass value="0.3"/>
+			<inertia ixx="0.005" ixy="0" ixz="0" iyy="0.005" iyz="0" izz="0.005"/>
 			<origin rpy="0 0 0" xyz="0.03536 -0.00072 -0.00207"/>
 		</inertial>
@@ -89,5 +89,5 @@
 		<inertial>
 			<mass value="0.0016579"/>
-			<inertia ixx="0.00156513" ixy="-1.47517e-05" ixz="-6.05746e-05" iyy="0.00173219" iyz="1.7619e-07" izz="0.000273081"/>
+			<inertia ixx="0.00156513" ixy="0" ixz="0" iyy="0.00173219" iyz="0" izz="0.000273081"/>
 		</inertial>
 	</link>
@@ -102,5 +102,5 @@
 		<inertial>
 			<mass value="0.3125"/>
-			<inertia ixx="0.000361198" ixy="1.98347e-06" ixz="6.35907e-07" iyy="0.000137229" iyz="5.68878e-06" izz="0.000399194"/>
+			<inertia ixx="0.000361198" ixy="0" ixz="0" iyy="0.000137229" iyz="0" izz="0.000399194"/>
 			<origin rpy="0 0 0" xyz="0.00018 0.01856 0.00099"/>
 		</inertial>
@@ -117,5 +117,5 @@
 		<inertial>
 			<mass value="0.50527"/>
-			<inertia ixx="0.000500872" ixy="3.55918e-05" ixz="8.51263e-05" iyy="0.00126284" iyz="-9.06813e-06" izz="0.00115718"/>
+			<inertia ixx="0.000500872" ixy="0" ixz="0" iyy="0.00126284" iyz="0" izz="0.00115718"/>
 			<origin rpy="0 0 0" xyz="0.08151 -0.01284 -0.01017"/>
 		</inertial>
@@ -132,5 +132,5 @@
 		<inertial>
 			<mass value="0.27495"/>
-			<inertia ixx="0.000122971" ixy="-9.86024e-07" ixz="-2.55838e-05" iyy="0.000331766" iyz="1.98925e-06" izz="0.000303047"/>
+			<inertia ixx="0.000122971" ixy="0" ixz="0" iyy="0.000331766" iyz="0" izz="0.000303047"/>
 			<origin rpy="0 0 0" xyz="-0.02297 0.00019 0.00119"/>
 		</inertial>
@@ -147,5 +147,5 @@
 		<inertial>
 			<mass value="0.16579"/>
-			<inertia ixx="0.00156513" ixy="-1.47517e-05" ixz="-6.05746e-05" iyy="0.00173219" iyz="1.7619e-07" izz="0.000273081"/>
+			<inertia ixx="0.00156513" ixy="0" ixz="0" iyy="0.00173219" iyz="0" izz="0.000273081"/>
 			<origin rpy="0 0 0" xyz="0.0593 -0.00271 -0.01014"/>
 		</inertial>
@@ -161,6 +161,6 @@
 	<link name="r_wrist">
 		<inertial>
-			<mass value="0.27555"/>
-			<inertia ixx="0.00156513" ixy="-1.47517e-05" ixz="-6.05746e-05" iyy="0.00173219" iyz="1.7619e-07" izz="0.000273081"/>
+			<mass value="0.3"/>
+			<inertia ixx="0.005" ixy="0" ixz="0" iyy="0.005" iyz="0" izz="0.005"/>
 			<origin rpy="0 0 0" xyz="0.03536 0.00072 -0.00207"/>
 		</inertial>
@@ -177,5 +177,5 @@
 		<inertial>
 			<mass value="0.0016579"/>
-			<inertia ixx="0.00156513" ixy="-1.47517e-05" ixz="-6.05746e-05" iyy="0.00173219" iyz="1.7619e-07" izz="0.000273081"/>
+			<inertia ixx="0.00156513" ixy="0" ixz="0" iyy="0.00173219" iyz="0" izz="0.000273081"/>
 		</inertial>
 	</link>
